File: Buttons.kicad_sch (KiCad schematic)
At the start: 21 parts

Commit message: modifications
Parts:
- added SW_mystery1: SW_mystery??, Button_Switch_SMD:SW_SPST_CK_RS282G05A3, symbol PCM_marbastlib-choc:choc_SW_HS
Connections:
- net GND: now also SW_mystery1.2
- new net SW_mystery: SW_mystery1.1
Changed lines of the file:
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@@
   (junction (at 46.736 39.116) (diameter 0) (color 0 0 0 0)
   )
+  (wire (pts (xy 83.82 88.9) (xy 92.71 88.9))
+    (stroke (width 0) (type default))
+  )
   (wire (pts (xy 107.95 39.37) (xy 117.475 39.37))
     (stroke (width 0) (type default))
@@
     (stroke (width 0) (type default))
   )
+  (wire (pts (xy 92.71 88.9) (xy 92.71 91.44))
+    (stroke (width 0) (type default))
+  )
+  (wire (pts (xy 73.66 83.82) (xy 78.74 83.82))
+    (stroke (width 0) (type default))
+  )
   (wire (pts (xy 107.95 27.94) (xy 116.84 27.94))
     (stroke (width 0) (type default))
@@
   (wire (pts (xy 117.475 39.37) (xy 126.365 39.37))
     (stroke (width 0) (type default))
+  )
+  (global_label "SW_mystery" (shape input) (at 73.66 83.82 180) (fields_autoplaced)
+    (effects (font (size 1.27 1.27)) (justify right))
+    (property "Intersheetrefs" "${INTERSHEET_REFS}" (at 59.7892 83.82 0)
+      (effects (font (size 1.27 1.27)) (justify right) hide)
+    )
   )
   (global_label "C_RT" (shape input) (at 106.045 62.23 90) (fields_autoplaced)
@@
     )
   )
+  (symbol (lib_id "PCM_marbastlib-choc:choc_SW_HS") (at 81.28 86.36 0) (unit 1)
+    (in_bom yes) (on_board yes) (dnp no)
+    (property "Reference" "SW_mystery1" (at 82.804 82.296 0)
+      (effects (font (size 1.27 1.27)))
+    )
+    (property "Value" "SW_mystery??" (at 81.28 82.042 0)
+      (effects (font (size 1.27 1.27)) hide)
+    )
+    (property "Footprint" "Button_Switch_SMD:SW_SPST_CK_RS282G05A3" (at 81.28 86.36 0)
+      (effects (font (size 1.27 1.27)) hide)
+    )
+    (property "Datasheet" "~" (at 81.28 86.36 0)
+      (effects (font (size 1.27 1.27)) hide)
+    )
+    (property "JLCPCB Part #" "C5117870" (at 81.28 86.36 0)
+      (effects (font (size 1.27 1.27)) hide)
+    )
+    (pin "1")
+    (pin "2")
+    (instances
+      (project "GRAM-SLIM"
+        (path "/17c378e5-d065-46dd-aa4a-654e3a402061/a547617f-d0d9-417f-8421-9ae0a9a5987b"
+          (reference "SW_mystery1") (unit 1)
+        )
+      )
+    )
+  )
   (symbol (lib_id "power:GND") (at 110.49 54.61 90) (unit 1)
     (in_bom yes) (on_board yes) (dnp no) (fields_autoplaced)
@@
         )
       )
+    )
+  )
+  (symbol (lib_id "power:GND") (at 92.71 91.44 0) (mirror y) (unit 1)
+    (in_bom yes) (on_board yes) (dnp no)
+    (property "Reference" "#PWR040" (at 92.71 97.79 0)
+      (effects (font (size 1.27 1.27)) hide)
+    )
+    (property "Value" "GND" (at 92.71 96.52 0)
+      (effects (font (size 1.27 1.27)))
+    )
+    (property "Footprint" "" (at 92.71 91.44 0)
+      (effects (font (size 1.27 1.27)) hide)
+    )
+    (property "Datasheet" "" (at 92.71 91.44 0)
+      (effects (font (size 1.27 1.27)) hide)
+    )
+    (pin "1")
+    (instances
+      (project "GRAM-SLIM"
+        (path "/17c378e5-d065-46dd-aa4a-654e3a402061/a547617f-d0d9-417f-8421-9ae0a9a5987b"
+          (reference "#PWR040") (unit 1)
+        )
+      )
