File: GRAM-SLIM.kicad_pcb (KiCad board)
At the start: 2 copper layers, 288.8 x 160.1 mm, 64 parts, among them J1 USB C Connector, J2 JTAG_TC2030, SW1 Boot, U1 XC6206, U2 USBLC6-2SC6, U3 RP2040, U4 W25Q128JVS, Y1 12MHz

Commit message: modifications
Parts:
- added SW_mystery1: SW_mystery??, Button_Switch_SMD:SW_SPST_CK_RS282G05A3, F.Cu at (102.0, 134.0)
Connections:
- U3 pad 14: unconnected-(U3-GPIO11-Pad14) -> SW_mystery
Routing:
- net SW_mystery: track 0.00 -> 167.6 mm, vias 0 -> 3
Other:
- outline, holes or cut-outs redrawn
