File: GRAM-SLIM.kicad_sch (KiCad schematic)
At the start: 42 parts, among them J1 USB C Connector, J2 JTAG_TC2030, SW1 Boot, U1 XC6206, U2 USBLC6-2SC6, U3 RP2040, U4 W25Q128JVS, Y1 12MHz

Commit message: modifications
Connections:
- net SW_mystery: now reaches U3.14 (GPIO11)
- no-connect marks 11 -> 10
Changed lines of the file:
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@@
   (no_connect (at 71.7108 74.168))
   (no_connect (at 71.7108 71.628))
-  (no_connect (at 71.7108 76.708))
   (no_connect (at 71.7108 107.188))
   (no_connect (at 129.54 51.816))
   (no_connect (at 71.7108 126.238))
+  (wire (pts (xy 72.39 76.2) (xy 72.39 76.708))
+    (stroke (width 0) (type default))
+  )
   (wire (pts (xy 64.516 164.084) (xy 64.516 165.354))
     (stroke (width 0) (type default))
@@
     (stroke (width 1) (type default))
   )
+  (wire (pts (xy 72.39 76.708) (xy 71.7108 76.708))
+    (stroke (width 0) (type default))
+  )
   (wire (pts (xy 70.866 164.084) (xy 70.866 165.354))
     (stroke (width 0) (type default))
@@
     (stroke (width 0) (type dash_dot_dot))
   )
+  (wire (pts (xy 73.66 76.2) (xy 72.39 76.2))
+    (stroke (width 0) (type default))
+  )
   (wire (pts (xy 102.997 134.874) (xy 104.267 134.874))
     (stroke (width 0) (type default))
@@
     )
   )
+  (global_label "SW_mystery" (shape bidirectional) (at 73.66 76.2 0) (fields_autoplaced)
+    (effects (font (size 1.27 1.27)) (justify left))
+    (property "Intersheetrefs" "${INTERSHEET_REFS}" (at 88.6421 76.2 0)
+      (effects (font (size 1.27 1.27)) (justify left) hide)
+    )
+  )
